File: XIAO ESP32S3 IMU.kicad_sch (KiCad schematic)
At the start: 9 parts, among them J2 Pins1_7, J3 Pins8_14, U1 Seeed Studio XIAO SAMD21, U2 MPU-9250

Commit message: gerber generation
Connections:
- net 3V3: now also J3.3 (Pin_3); no longer J3.5 (Pin_5)
- net FSYNC: now also J3.5 (Pin_5); no longer J3.3 (Pin_3)
- net GND: now also J3.2 (Pin_2); no longer J3.6 (Pin_6)
Other:
- moved on the sheet: J3
Changed lines of the file:
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@@
     )
   )
-  (symbol (lib_id "Connector:Conn_01x07_Socket") (at 149.86 79.375 180) (unit 1)
+  (symbol (lib_id "Connector:Conn_01x07_Socket") (at 149.86 79.375 0) (mirror y) (unit 1)
     (in_bom yes) (on_board yes) (dnp no)
-    (property "Reference" "J3" (at 148.59 80.645 0)
+    (property "Reference" "J3" (at 148.59 78.105 0)
       (effects (font (size 1.27 1.27)) (justify left))
     )
-    (property "Value" "Pins8_14" (at 148.59 78.105 0)
+    (property "Value" "Pins8_14" (at 148.59 80.645 0)
       (effects (font (size 1.27 1.27)) (justify left))
     )
